Commit message: added camera link to xacro file

File: dvrk_model/model/ecm.urdf.xacro (robot description, xacro)
@@ -5,4 +5,5 @@
   <!-- Macro for da Vinci Endoscope Camera Manipulator (ECM) -->
   <xacro:macro name="ecm" params="prefix parent_link xyz rpy">
+  <xacro:property name="cameraSize" value="0.05"/>
     <!-- Joint 0: Fixed to World-->
     <joint name="setup_fixed_joint" type="fixed">
@@ -205,4 +206,28 @@
       </collision>
     </link>
+    <!-- Camera -->
+    <joint name="camera joint" type="fixed">
+      <parent link="${prefix}_roll_link"/>
+      <child link="camera"/>
+      <origin rpy="0 0 0" xyz="0 0 0"/>
+      <axis xyz="0 0 1"/>
+      <joint_properties damping="1.0" friction="0.0"/>
+      <limit effort="100.0" lower="-${PI/2}" upper="${PI/2}" velocity="10"/>
+    </joint>
+   <link name="camera">
+	<visual>
+    	    <origin rpy="0 0 0" xyz="0.0 0 0"/>
+    	    <geometry>
+      	    <box size="${cameraSize} ${cameraSize} ${cameraSize}"/>
+    	    </geometry>
+       	    <material name="blue"/>
+  	</visual>
+	<collision>
+    	    <origin rpy="0 0 0" xyz="0.0 0 0"/>
+    	    <geometry>
+      	    <box size="${cameraSize} ${cameraSize} ${cameraSize}"/>
+    	    </geometry>
+  	</collision>
+    </link>
   </xacro:macro>
 </robot>

Commit message: added cube in the foreground directed to ECM urdf

File: dvrk_model/model/ecm.urdf.xacro (robot description, xacro)
@@ -210,5 +210,5 @@
       <parent link="${prefix}_roll_link"/>
       <child link="camera"/>
-      <origin rpy="0 0 0" xyz="0 0 0"/>
+      <origin rpy="0 0 ${PI/2}" xyz="0 0 0"/>
       <axis xyz="0 0 1"/>
       <joint_properties damping="1.0" friction="0.0"/>
@@ -219,5 +219,5 @@
     	    <origin rpy="0 0 0" xyz="0.0 0 0"/>
     	    <geometry>
-      	    <box size="${cameraSize} ${cameraSize} ${cameraSize}"/>
+      	      <cylinder length="0.06" radius="0.02"/>
     	    </geometry>
        	    <material name="blue"/>
@@ -226,8 +226,25 @@
     	    <origin rpy="0 0 0" xyz="0.0 0 0"/>
     	    <geometry>
-      	    <box size="${cameraSize} ${cameraSize} ${cameraSize}"/>
+      	      <cylinder length="0.06" radius="0.02"/>
     	    </geometry>
   	</collision>
     </link>
+    <!-- Cube object with dVRK logo -->
+    <joint name="cube_joint" type="fixed">
+	<parent link="${parent_link}"/>
+	<child link="cube_object"/>
+        <origin rpy="0 0 0" xyz="0.5 0 -1"/>
+        <axis xyz="0 0 1"/>
+    </joint>
+    <link name="cube_object">
+      <visual>
+        <origin rpy="0.0 0 0" xyz="0 0 0"/>
+        <geometry>
+          <!-- <mesh filename="package://dvrk_model/meshes/dVRK-cube.stl" scale="2 2 2"/>-->
+	  <box size="0.1 0.05 0.05"/>
+          <material name="DaVinciBlue"/>
+        </geometry>
+      </visual>
+    </link>
   </xacro:macro>
 </robot>
